Commit message: Path Planning Demo

File: isaac_sim_assets/urdf_isaac_sim/kuka_description/urdf/kuka_description.urdf (robot description, URDF)
Before this commit: robot kuka, 7 links, 6 joints
Links:
- link base_link: geometry collision mesh filename=/home/one/palletizing_project/isaac_sim_assets/urdf_isaac_s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; visual mesh filename=/home/one/palletizing_project/isaac_sim_assets/urdf_isaac_s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
- link link_1: geometry collision mesh filename=/home/one/palletizing_project/isaac_sim_assets/urdf_isaac_s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; visual mesh filename=/home/one/palletizing_project/isaac_sim_assets/urdf_isaac_s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
- link link_2: geometry collision mesh filename=/home/one/palletizing_project/isaac_sim_assets/urdf_isaac_s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; visual mesh filename=/home/one/palletizing_project/isaac_sim_assets/urdf_isaac_s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
- link link_3: geometry collision mesh filename=/home/one/palletizing_project/isaac_sim_assets/urdf_isaac_s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; visual mesh filename=/home/one/palletizing_project/isaac_sim_assets/urdf_isaac_s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
- link link_4: geometry collision mesh filename=/home/one/palletizing_project/isaac_sim_assets/urdf_isaac_s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; visual mesh filename=/home/one/palletizing_project/isaac_sim_assets/urdf_isaac_s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
- link link_5: geometry collision mesh filename=/home/one/palletizing_project/isaac_sim_assets/urdf_isaac_s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; visual mesh filename=/home/one/palletizing_project/isaac_sim_assets/urdf_isaac_s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
- link link_6: geometry collision mesh filename=/home/one/palletizing_project/isaac_sim_assets/urdf_isaac_s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; visual mesh filename=/home/one/palletizing_project/isaac_sim_assets/urdf_isaac_s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

File: kuka_ws/src/kuka_description/urdf/kuka_description.urdf (robot description, URDF)
Before this commit: robot kuka, 7 links, 6 joints
Joints:
- joint joint6: limit lower=-6.1086523819801535 upper=6.1086523819801535 effort=0 velocity=6.283185307179586 -> lower=-3.1416 upper=3.1416 effort=0 velocity=6.283185307179586
