Commit message: Update KUKA 4DOF moveit configs and palletizing server logic

File: kuka_ws/src/kuka_moveit_config/config/assembly_moveit.ros2_control.xacro (robot description, xacro)
@@ -3,8 +3,9 @@
     <xacro:macro name="assembly_moveit_ros2_control" params="name initial_positions_file">
         <xacro:property name="initial_positions" value="${load_yaml(initial_positions_file)['initial_positions']}"/>
-        <!-- <ros2_control name="${name}" type="system">
-            <hardware> -->
-                <!-- By default, set up controllers for simulation. This won't work on real hardware -->
-                <!-- <plugin>mock_components/GenericSystem</plugin>
+        <ros2_control name="${name}" type="system">
+            <hardware>
+                <plugin>mock_components/GenericSystem</plugin>
+                <param name="mock_sensor_commands">false</param>
+                <param name="state_following_offset">0.0</param>
             </hardware>
             <joint name="joint1">
@@ -50,5 +51,7 @@
                 <state_interface name="velocity"/>
             </joint>
-        </ros2_control> -->
+        </ros2_control>
+    </xacro:macro>
+    <xacro:macro name="assembly_moveit_ros2_control_isaac" params="name">
         <ros2_control name="IsaacSimSystem" type="system">
             <hardware>

File: kuka_ws/src/kuka_moveit_config/config/assembly_moveit.urdf.xacro (robot description, xacro)
@@ -2,8 +2,14 @@
 <robot xmlns:xacro="http://www.ros.org/wiki/xacro" name="assembly_moveit">
     <xacro:arg name="initial_positions_file" default="initial_positions.yaml" />
+    <xacro:arg name="use_isaac_sim" default="false" />
     <!-- Import assembly_moveit urdf file -->
     <xacro:include filename="$(find kuka_description)/urdf/assembly_moveit.xacro" />
     <!-- Import control_xacro -->
     <xacro:include filename="assembly_moveit.ros2_control.xacro" />
-    <xacro:assembly_moveit_ros2_control name="FakeSystem" initial_positions_file="$(arg initial_positions_file)"/>
+    <xacro:if value="$(arg use_isaac_sim)">
+        <xacro:assembly_moveit_ros2_control_isaac name="IsaacSimSystem"/>
+    </xacro:if>
+    <xacro:unless value="$(arg use_isaac_sim)">
+        <xacro:assembly_moveit_ros2_control name="FakeSystem" initial_positions_file="$(arg initial_positions_file)"/>
+    </xacro:unless>
 </robot>
